Commit message: Small changes

File: src/ur3e_description/urdf/onrobot_2fg7.xacro (robot description, xacro)
@@ -4,4 +4,5 @@
   <xacro:include filename="$(find ur3e_description)/urdf/materials.xacro" />
   <xacro:macro name="onrobot_2fg7" params="prefix parent *origin">
+    <xacro:property name="fixed_grip_offset" value="0.02" />
     <link name="${prefix}base_link">
       <inertial>
@@ -26,19 +27,13 @@
     <link name="${prefix}right_attachment"></link>
     <link name="${prefix}left_attachment"></link>
-    <joint name="${prefix}gripper_joint" type="prismatic">
-      <origin xyz="0.0 0.0 0.11" rpy="0 0 0" />
+    <joint name="${prefix}gripper_joint" type="fixed">
+      <origin xyz="-${fixed_grip_offset} 0.0 0.11" rpy="0 0 0" />
       <parent link="${prefix}base_link" />
       <child link="${prefix}left_attachment" />
-      <axis xyz="-1.0 0.0 0.0" />
-      <limit lower="0.0115" upper="0.0305" effort="140" velocity="0.45" />
-      <!-- total 0.38 -->
     </joint>
-    <joint name="${prefix}right_finger_joint" type="prismatic">
-      <origin xyz="0.0 0.0 0.11" rpy="0 0 0" />
+    <joint name="${prefix}right_finger_joint" type="fixed">
+      <origin xyz="${fixed_grip_offset} 0.0 0.11" rpy="0 0 0" />
       <parent link="${prefix}base_link" />
       <child link="${prefix}right_attachment" />
-      <axis xyz="1.0 0.0 0.0" />
-      <limit lower="0.0115" upper="0.0305" effort="140" velocity="0.45" />
-      <mimic joint="${prefix}gripper_joint" multiplier="1.0" />
     </joint>
     <joint name="${prefix}2fg7_attach_joint" type="fixed">

Commit message: Wider gripper base

File: src/ur3e_description/urdf/onrobot_2fg7.xacro (robot description, xacro)
@@ -5,4 +5,7 @@
   <xacro:macro name="onrobot_2fg7" params="prefix parent *origin">
     <xacro:property name="fixed_grip_offset" value="0.02" />
+    <xacro:property name="base_width" value="0.09" />
+    <xacro:property name="base_depth" value="0.075" />
+    <xacro:property name="base_height" value="0.11" />
     <link name="${prefix}base_link">
       <inertial>
@@ -14,5 +17,5 @@
         <origin xyz="0 0 0.055" rpy="0 0 0" />
         <geometry>
-          <box size="0.055 0.075 0.11" />
+          <box size="${base_width} ${base_depth} ${base_height}" />
         </geometry>
         <material name="silver" />
@@ -21,5 +24,5 @@
         <origin xyz="0 0 0.055" rpy="0 0 0" />
         <geometry>
-          <box size="0.055 0.075 0.11" />
+          <box size="${base_width} ${base_depth} ${base_height}" />
         </geometry>
       </collision>
