Commit message: Update UR3e cell model with better gripper/camera

File: src/ur3e_description/urdf/ur3e_cell.urdf.xacro (robot description, xacro)
@@ -1,40 +1,46 @@
 <?xml version="1.0"?>
 <robot xmlns:xacro="http://wiki.ros.org/xacro" name="ur3e_cell">
-  <xacro:include filename="$(find ur_description)/urdf/ur_macro.xacro"/>
-  <xacro:include filename="$(find ur_robot_driver)/urdf/ur.ros2_control.xacro"/>
-  <xacro:include filename="$(find ur_description)/urdf/inc/ur_transmissions.xacro"/>
-  <xacro:property name="robot_name" value="ur"/>
-  <xacro:property name="tf_prefix" value=""/>
-  <xacro:property name="joint_limit_params" value="$(find ur_description)/config/ur3e/joint_limits.yaml"/>
-  <xacro:property name="kinematics_params" value="$(find ur_description)/config/ur3e/default_kinematics.yaml"/>
-  <xacro:property name="physical_params" value="$(find ur_description)/config/ur3e/physical_parameters.yaml"/>
-  <xacro:property name="visual_params" value="$(find ur_description)/config/ur3e/visual_parameters.yaml"/>
-  <xacro:property name="transmission_hw_interface" value=""/>
-  <xacro:property name="safety_limits" value="false"/>
-  <xacro:property name="safety_pos_margin" value="0.15"/>
-  <xacro:property name="safety_k_position" value="20"/>
-  <xacro:property name="headless_mode" value="false"/>
-  <xacro:property name="robot_ip" value="0.0.0.0"/>
-  <xacro:property name="script_filename" value=""/>
-  <xacro:property name="output_recipe_filename" value=""/>
-  <xacro:property name="input_recipe_filename" value=""/>
-  <xacro:property name="reverse_ip" value="0.0.0.0"/>
-  <xacro:property name="script_command_port" value="50004"/>
-  <xacro:property name="reverse_port" value="50001"/>
-  <xacro:property name="script_sender_port" value="50002"/>
-  <xacro:property name="trajectory_port" value="50003"/>
-  <xacro:property name="use_tool_communication" value="false"/>
-  <xacro:property name="tool_voltage" value="0"/>
-  <xacro:property name="tool_parity" value="0"/>
-  <xacro:property name="tool_baud_rate" value="115200"/>
-  <xacro:property name="tool_stop_bits" value="1"/>
-  <xacro:property name="tool_rx_idle_chars" value="1.5"/>
-  <xacro:property name="tool_tx_idle_chars" value="3.5"/>
-  <xacro:property name="tool_device_name" value="/tmp/ttyUR"/>
-  <xacro:property name="tool_tcp_port" value="54321"/>
-  <xacro:property name="use_mock_hardware" value="false"/>
-  <xacro:property name="mock_sensor_commands" value="false"/>
-  <xacro:property name="initial_positions_file" value="$(find ur_description)/config/initial_positions.yaml"/>
-  <link name="world"/>
+  <xacro:include filename="$(find ur_description)/urdf/ur_macro.xacro" />
+  <xacro:include filename="$(find ur_robot_driver)/urdf/ur.ros2_control.xacro" />
+  <xacro:include filename="$(find ur_description)/urdf/inc/ur_transmissions.xacro" />
+  <xacro:include filename="$(find ur3e_description)/urdf/onrobot_2fg7.xacro" />
+  <xacro:property name="robot_name" value="ur" />
+  <xacro:property name="tf_prefix" value="" />
+  <xacro:property name="joint_limit_params"
+    value="$(find ur_description)/config/ur3e/joint_limits.yaml" />
+  <xacro:property name="kinematics_params"
+    value="$(find ur_description)/config/ur3e/default_kinematics.yaml" />
+  <xacro:property name="physical_params"
+    value="$(find ur_description)/config/ur3e/physical_parameters.yaml" />
+  <xacro:property name="visual_params"
+    value="$(find ur_description)/config/ur3e/visual_parameters.yaml" />
+  <xacro:property name="transmission_hw_interface" value="" />
+  <xacro:property name="safety_limits" value="false" />
+  <xacro:property name="safety_pos_margin" value="0.15" />
+  <xacro:property name="safety_k_position" value="20" />
+  <xacro:property name="headless_mode" value="false" />
+  <xacro:property name="robot_ip" value="0.0.0.0" />
+  <xacro:property name="script_filename" value="" />
+  <xacro:property name="output_recipe_filename" value="" />
+  <xacro:property name="input_recipe_filename" value="" />
+  <xacro:property name="reverse_ip" value="0.0.0.0" />
+  <xacro:property name="script_command_port" value="50004" />
+  <xacro:property name="reverse_port" value="50001" />
+  <xacro:property name="script_sender_port" value="50002" />
+  <xacro:property name="trajectory_port" value="50003" />
+  <xacro:property name="use_tool_communication" value="false" />
+  <xacro:property name="tool_voltage" value="0" />
+  <xacro:property name="tool_parity" value="0" />
+  <xacro:property name="tool_baud_rate" value="115200" />
+  <xacro:property name="tool_stop_bits" value="1" />
+  <xacro:property name="tool_rx_idle_chars" value="1.5" />
+  <xacro:property name="tool_tx_idle_chars" value="3.5" />
+  <xacro:property name="tool_device_name" value="/tmp/ttyUR" />
+  <xacro:property name="tool_tcp_port" value="54321" />
+  <xacro:property name="use_mock_hardware" value="false" />
+  <xacro:property name="mock_sensor_commands" value="false" />
+  <xacro:property name="initial_positions_file"
+    value="$(find ur_description)/config/initial_positions.yaml" />
+  <link name="world" />
   <xacro:ur_robot
     name="${robot_name}"
@@ -48,60 +54,46 @@
     safety_pos_margin="${safety_pos_margin}"
     safety_k_position="${safety_k_position}">
-    <origin xyz="0 0 0" rpy="0 0 0"/>
+    <origin xyz="0 0 0" rpy="0 0 0" />
   </xacro:ur_robot>
-  <!--
-    Placeholder geometry for collision-aware planning.
-    Adjust sizes and offsets to roughly match your real setup.
-    These links are fixed to the robot, so MoveIt will treat them as part of the arm.
-  -->
-  <link name="${tf_prefix}gripper_body">
+  <xacro:onrobot_2fg7 prefix="${tf_prefix}gripper_" parent="${tf_prefix}tool0">
+    <origin xyz="0 0 0" rpy="0 0 0" />
+  </xacro:onrobot_2fg7>
+  <xacro:onrobot_2fg7_fingertip
+    prefix="${tf_prefix}gripper_right_"
+    parent="${tf_prefix}gripper_right_attachment">
+    <origin xyz="0 0 0" rpy="0 0 3.14159265359" />
+  </xacro:onrobot_2fg7_fingertip>
+  <xacro:onrobot_2fg7_fingertip
+    prefix="${tf_prefix}gripper_left_"
+    parent="${tf_prefix}gripper_left_attachment">
+    <origin xyz="0 0 0" rpy="0 0 0" />
+  </xacro:onrobot_2fg7_fingertip>
+  <link name="${tf_prefix}camera_body">
     <visual>
-      <origin xyz="0 0 0.08" rpy="0 0 0"/>
+      <origin xyz="0 0.03 0.015" rpy="0 0 0" />
       <geometry>
-        <box size="0.06 0.06 0.16"/>
+        <box size="0.06 0.075 0.03" />
       </geometry>
-      <material name="gripper_gray">
-        <color rgba="0.45 0.45 0.45 1.0"/>
+      <material name="camera_blue">
+        <color rgba="0.15 0.35 0.8 1.0" />
       </material>
     </visual>
     <collision>
-      <origin xyz="0 0 0.08" rpy="0 0 0"/>
+      <origin xyz="0 0.03 0.015" rpy="0 0 0" />
       <geometry>
-        <box size="0.06 0.06 0.16"/>
+        <box size="0.06 0.075 0.03" />
       </geometry>
     </collision>
   </link>
-  <joint name="${tf_prefix}tool0-gripper_body" type="fixed">
-    <parent link="${tf_prefix}tool0"/>
-    <child link="${tf_prefix}gripper_body"/>
-    <origin xyz="0 0 0.02" rpy="0 0 0"/>
+  <joint name="${tf_prefix}gripper_base_link-camera_body" type="fixed">
+    <parent link="${tf_prefix}gripper_base_link" />
+    <child link="${tf_prefix}camera_body" />
+    <origin xyz="0 0.0315 -0.0125" rpy="0 0 0" />
   </joint>
-  <link name="${tf_prefix}camera_body">
-    <visual>
-      <origin xyz="0.045 0 0.015" rpy="0 0 0"/>
-      <geometry>
-        <box size="0.09 0.03 0.03"/>
-      </geometry>
-      <material name="camera_blue">
-        <color rgba="0.15 0.35 0.8 1.0"/>
-      </material>
-    </visual>
-    <collision>
-      <origin xyz="0.045 0 0.015" rpy="0 0 0"/>
-      <geometry>
-        <box size="0.09 0.03 0.03"/>
-      </geometry>
-    </collision>
-  </link>
-  <joint name="${tf_prefix}gripper_body-camera_body" type="fixed">
-    <parent link="${tf_prefix}gripper_body"/>
-    <child link="${tf_prefix}camera_body"/>
-    <origin xyz="0.025 0 0.11" rpy="0 0 0"/>
-  </joint>
-  <link name="${tf_prefix}camera_frame"/>
+  <link name="${tf_prefix}camera_frame" />
   <joint name="${tf_prefix}camera_body-camera_frame" type="fixed">
-    <parent link="${tf_prefix}camera_body"/>
-    <child link="${tf_prefix}camera_frame"/>
-    <origin xyz="0 0 0" rpy="0 0 0"/>
+    <parent link="${tf_prefix}camera_body" />
+    <child link="${tf_prefix}camera_frame" />
+    <origin xyz="0 0 0" rpy="0 0 0" />
   </joint>
   <xacro:ur_ros2_control

Commit message: Improve MoveIt pick pipeline

File: src/ur3e_description/urdf/ur3e_cell.urdf.xacro (robot description, xacro)
@@ -69,4 +69,10 @@
     <origin xyz="0 0 0" rpy="0 0 0" />
   </xacro:onrobot_2fg7_fingertip>
+  <link name="${tf_prefix}gripper_tcp" />
+  <joint name="${tf_prefix}gripper_base_link-gripper_tcp" type="fixed">
+    <parent link="${tf_prefix}gripper_base_link" />
+    <child link="${tf_prefix}gripper_tcp" />
+    <origin xyz="0 0 0.15" rpy="0 0 0" />
+  </joint>
   <link name="${tf_prefix}camera_body">
     <visual>

Commit message: Add table

File: src/ur3e_description/urdf/ur3e_cell.urdf.xacro (robot description, xacro)
@@ -43,4 +43,16 @@
     default="$(find ur_description)/config/initial_positions.yaml" />
   <link name="world" />
+  <link name="table">
+    <collision>
+      <geometry>
+        <box size="1.0 1.0 0.04" />
+      </geometry>
+    </collision>
+  </link>
+  <joint name="world-table" type="fixed">
+    <parent link="world" />
+    <child link="table" />
+    <origin xyz="0 0 -0.03" rpy="0 0 0" />
+  </joint>
   <xacro:ur_robot
     name="$(arg name)"

Commit message: Add camera mount collision box to the urdf

File: src/ur3e_description/urdf/ur3e_cell.urdf.xacro (robot description, xacro)
@@ -103,4 +103,19 @@
       </geometry>
     </collision>
+    <visual>
+      <origin xyz="0 -0.03 0.0" rpy="0 0 0" />
+      <geometry>
+        <box size="0.09 0.10 0.06" />
+      </geometry>
+      <material name="camera_mount">
+        <color rgba="0.85 0.25 0.25 0.45" />
+      </material>
+    </visual>
+    <collision>
+      <origin xyz="0 -0.03 0.0" rpy="0 0 0" />
+      <geometry>
+        <box size="0.09 0.10 0.06" />
+      </geometry>
+    </collision>
   </link>
   <joint name="$(arg tf_prefix)gripper_base_link-camera_body" type="fixed">

Commit message: Small fixes

File: src/ur3e_description/urdf/ur3e_cell.urdf.xacro (robot description, xacro)
@@ -104,7 +104,7 @@
     </collision>
     <visual>
-      <origin xyz="0 -0.03 0.0" rpy="0 0 0" />
+      <origin xyz="0 -0.0225 0.0" rpy="0 0 0" />
       <geometry>
-        <box size="0.09 0.10 0.06" />
+        <box size="0.12 0.115 0.06" />
       </geometry>
       <material name="camera_mount">
@@ -113,7 +113,7 @@
     </visual>
     <collision>
-      <origin xyz="0 -0.03 0.0" rpy="0 0 0" />
+      <origin xyz="0 -0.0225 0.0" rpy="0 0 0" />
       <geometry>
-        <box size="0.09 0.10 0.06" />
+        <box size="0.12 0.115 0.06" />
       </geometry>
     </collision>

Commit message: Small adjustments

File: src/ur3e_description/urdf/ur3e_cell.urdf.xacro (robot description, xacro)
@@ -89,7 +89,7 @@
   <link name="$(arg tf_prefix)camera_body">
     <visual>
-      <origin xyz="0 0.03 0.015" rpy="0 0 0" />
+      <origin xyz="0 0.0375 0.015" rpy="0 0 0" />
       <geometry>
-        <box size="0.06 0.075 0.03" />
+        <box size="0.06 0.09 0.03" />
       </geometry>
       <material name="camera_blue">
@@ -98,7 +98,7 @@
     </visual>
     <collision>
-      <origin xyz="0 0.03 0.015" rpy="0 0 0" />
+      <origin xyz="0 0.0375 0.015" rpy="0 0 0" />
       <geometry>
-        <box size="0.06 0.075 0.03" />
+        <box size="0.06 0.09 0.03" />
       </geometry>
     </collision>
